Commit message: Rviz integration completed

File: src/my_robot/urdf/my_robot.xacro (robot description, xacro)
@@ -1,5 +1,5 @@
 <?xml version='1.0'?>
 <robot name="my_robot" xmlns:xacro="http://www.ros.org/wiki/xacro">
-  <link name="robot_footprint"></link>
+<link name="robot_footprint"></link>
 <xacro:include filename="$(find my_robot)/urdf/my_robot.gazebo" />
   <joint name="robot_footprint_joint" type="fixed">
@@ -9,5 +9,5 @@
   </joint>
   <link name='chassis'>
-    <pose>0 0 0.1 0 0 0</pose>
+    <pose xyz="0 0 0.1" rpy=" 0 0 0"/>
     <inertial>
       <mass value="15.0"/>
@@ -22,5 +22,5 @@
       <origin xyz="0 0 0" rpy=" 0 0 0"/>
       <geometry>
-        <box size=".4 .2 .1"/>
+        <box size="0.4 0.2 0.1"/>
       </geometry>
     </collision>
@@ -28,5 +28,5 @@
       <origin xyz="0 0 0" rpy=" 0 0 0"/>
       <geometry>
-        <box size=".4 .2 .1"/>
+  <box size="0.4 0.2 0.1"/>
       </geometry>
     </visual>
@@ -83,5 +83,5 @@
     <child link="left_wheel"/>
     <parent link="chassis"/>
-    <axis xyz="0 1 0" rpy="0 0 0"/>
+    <axis xyz="0 1.0 0" rpy="0 0 0"/>
     <limit effort="10000" velocity="1000"/>
     <dynamics damping="1.0" friction="1.0"/>
@@ -114,5 +114,5 @@
     <child link="right_wheel"/>
     <parent link="chassis"/>
-    <axis xyz="0 1 0" rpy="0 0 0"/>
+    <axis xyz="0 1.0 0" rpy="0 0 0"/>
     <limit effort="10000" velocity="1000"/>
     <dynamics damping="1.0" friction="1.0"/>
@@ -130,13 +130,13 @@
     </inertial>
     <visual>
-      <geometry>
 	<origin xyz="0 0 0" rpy="0 0 0" />
-	<box size=".05 .05 .05"/>
+        <geometry>
+	<box size="0.05 0.05 0.05"/>
 	</geometry>
     </visual>
     <collision>
-      <geometry>
 	<origin xyz="0 0 0" rpy="0 0 0" />
-	<box size=".05 .05 .05"/>
+        <geometry>
+	<box size="0.05 0.05 0.05"/>
 	</geometry>
     </collision>
@@ -147,5 +147,5 @@
     <child link="camera"/>
     <parent link="chassis"/>
-    <axis xyz="0 1 0" rpy="0 0 0"/>
+    <axis xyz="0 1.0 0" rpy="0 0 0"/>
     <limit effort="10000" velocity="1000"/>
     <dynamics damping="1.0" friction="1.0"/>
@@ -169,7 +169,7 @@
     </visual>
     <collision>
+	<origin xyz="0 0 0" rpy="0 0 0" />
       <geometry>
-	<origin xyz="0 0 0" rpy="0 0 0" />
-	<box size=".1 .1 .1"/>
+	<box size="0.1 0.1 0.1"/>
 	</geometry>
     </collision>
@@ -180,5 +180,5 @@
     <child link="hokuyo"/>
     <parent link="chassis"/>
-    <axis xyz="0 1 0" rpy="0 0 0"/>
+    <axis xyz="0 1.0 0" rpy="0 0 0"/>
     <limit effort="10000" velocity="1000"/>
     <dynamics damping="1.0" friction="1.0"/>
